File: hardware/5v-power.kicad_pcb (KiCad board)
At the start: 4 copper layers, 100 x 50 mm, 110 parts, among them J1 Conn_01x04, J2 Screw_Terminal_01x02, J3 USB_A_Stacked, J4 USB_A_Stacked, J5 USB_A_Stacked, J6 USB_A_Stacked, J7 RJ45_Abracon_ARJM11D7-009-AB-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, J8 Conn_01x03_Pin, J9 Conn_01x03_Pin, Q1 AO3401A, Q10 AO3401A, Q11 MMBT3904, Q12 MMBT3904, Q13 AO3401A, Q14 AO3401A, Q15 MMBT3904, Q16 MMBT3904, Q2 AO3401A, Q3 MMBT3904, Q4 MMBT3904, Q5 AO3401A, Q6 AO3401A, Q7 MMBT3904, Q8 MMBT3904, Q9 AO3401A, U1 W5500, U2 INA4180, U3 INA4180, U4 AMS1117-3.3, U5 ATSAMD21G17A-M, Y1 RH100-25.000-18-F-1020-EXT-TR

Commit message: rev2
Parts:
- added D4: LED_Small, LED_SMD:LED_0603_1608Metric, B.Cu at (167.2, 122.5)
- added R49: R_Small, Resistor_SMD:R_0603_1608Metric, B.Cu at (167.2, 121.0)
- D1, D2, D3, R46, R5, R6: moved to B.Cu
- R14, R21, R28: value 5m -> 1M; footprint Resistor_SMD:R_0805_2012Metric -> Resistor_SMD:R_0603_1608Metric
- R19, R26, R3: value 1M -> 5m; footprint Resistor_SMD:R_0603_1608Metric -> Resistor_SMD:R_0805_2012Metric
- moved R4 29.2 mm to (98.2, 103.4), turned to 0 degrees
- moved R9 20.2 mm to (123.7, 103.3), turned to 0 degrees
- moved R3 13.5 mm to (120.2, 103.3), turned to 0 degrees
- moved R19 13.5 mm to (142.2, 103.3), turned to 0 degrees
- moved R26 13.4 mm to (164.2, 103.4), turned to 0 degrees
- moved R46 11.4 mm to (144.8, 121.0), turned to 0 degrees
- moved D3 11.2 mm to (144.7, 122.5), turned to 0 degrees
- moved R5 11.0 mm to (101.0, 120.9), turned to 0 degrees
- moved R6 10.9 mm to (123.1, 120.8), turned to 0 degrees
- moved R21 10.9 mm to (154.6, 110.9), turned to -90 degrees
- moved D1 10.8 mm to (100.9, 122.4), turned to 0 degrees
- moved D2 10.8 mm to (123.1, 122.4), turned to 0 degrees
- moved R14 10.7 mm to (132.7, 110.6), turned to -90 degrees
- moved R28 10.2 mm to (176.8, 109.7), turned to -90 degrees
- moved C9 6.90 mm to (157.8, 92.3), turned to 0 degrees
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Connections:
- J3 pad 1: Net-(J3-VBUS1) -> /port1_isense1-
- J3 pad 4: /port1_isense1 -> GND
- J3 pad 5: Net-(J3-VBUS2) -> /port1_isense2-
- J3 pad 8: /port1_isense2 -> GND
- J4 pad 1: Net-(J4-VBUS1) -> /port2_isense1-
- J4 pad 4: /port2_isense1+ -> GND
- J4 pad 5: Net-(J4-VBUS2) -> /port2_isense2-
- J4 pad 8: /port2_isense2+ -> GND
- J5 pad 1: Net-(J5-VBUS1) -> /port3_isense1-
- J5 pad 4: /port3_isense1 -> GND
- J5 pad 5: Net-(J5-VBUS2) -> /port3_isense2-
- J5 pad 8: /port3_isense2 -> GND
- J6 pad 1: Net-(J6-VBUS1) -> /port4_isense1-
- J6 pad 4: /port4_isense1+ -> GND
- J6 pad 5: Net-(J6-VBUS2) -> /port4_isense2-
- J6 pad 8: /port4_isense2+ -> GND
- Q1 pad 3: Net-(J3-VBUS1) -> /port1_isense1+
- Q10 pad 3: Net-(J5-VBUS2) -> /port3_isense2+
- Q13 pad 3: Net-(J6-VBUS1) -> /port4_isense1+
- Q14 pad 3: Net-(J6-VBUS2) -> /port4_isense2+
- Q2 pad 3: Net-(J3-VBUS2) -> /port1_isense2+
- Q5 pad 3: Net-(J4-VBUS1) -> /port2_isense1+
- Q6 pad 3: Net-(J4-VBUS2) -> /port2_isense2+
- Q9 pad 3: Net-(J5-VBUS1) -> /port3_isense1+
- R14 pad 1: /port2_isense2+ -> Net-(J4-Shield)
- R19 pad 1: Net-(J5-Shield) -> /port3_isense1-
- R19 pad 2: GND -> /port3_isense1+
- R20 pad 1: /port3_isense1 -> /port3_isense2-
- R20 pad 2: GND -> /port3_isense2+
- R21 pad 1: /port3_isense2 -> Net-(J5-Shield)
- R26 pad 1: Net-(J6-Shield) -> /port4_isense1-
- R26 pad 2: GND -> /port4_isense1+
- R27 pad 1: /port4_isense1+ -> /port4_isense2-
- R27 pad 2: GND -> /port4_isense2+
- R28 pad 1: /port4_isense2+ -> Net-(J6-Shield)
- R3 pad 1: Net-(J4-Shield) -> /port2_isense1-
- R3 pad 2: GND -> /port2_isense1+
- R4 pad 1: /port2_isense1+ -> /port1_isense1-
- R4 pad 2: GND -> /port1_isense1+
- R8 pad 1: /port1_isense1 -> /port1_isense2-
- R8 pad 2: GND -> /port1_isense2+
- R9 pad 1: /port1_isense2 -> /port2_isense2-
- R9 pad 2: GND -> /port2_isense2+
- U2 pad 1: /port1_isense2_out -> /port2_isense2_out
- U2 pad 10: /port2_isense2+ -> /port1_isense1+
- U2 pad 12: /port2_isense1+ -> /port1_isense2+
- U2 pad 13: GND -> /port1_isense2-
- U2 pad 14: /port2_isense1_out -> /port1_isense1_out
- U2 pad 2: GND -> /port2_isense1-
- U2 pad 3: /port1_isense2 -> /port2_isense1+
- U2 pad 5: /port1_isense1 -> /port2_isense2+
- U2 pad 6: GND -> /port2_isense2-
- U2 pad 7: /port1_isense1_out -> /port2_isense1_out
- U2 pad 8: /port2_isense2_out -> /port1_isense2_out
- U2 pad 9: GND -> /port1_isense1-
- U3 pad 1: /port3_isense2_out -> /port4_isense2_out
- U3 pad 10: /port4_isense2+ -> /port3_isense1+
- U3 pad 12: /port4_isense1+ -> /port3_isense2+
- U3 pad 13: GND -> /port3_isense2-
- U3 pad 14: /port4_isense1_out -> /port3_isense1_out
- U3 pad 2: GND -> /port4_isense1-
- U3 pad 3: /port3_isense2 -> /port4_isense1+
- U3 pad 5: /port3_isense1 -> /port4_isense2+
- U3 pad 6: GND -> /port4_isense2-
- U3 pad 7: /port3_isense1_out -> /port4_isense1_out
- U3 pad 8: /port4_isense2_out -> /port3_isense2_out
- U3 pad 9: GND -> /port3_isense1-
- U5 pad 32: unconnected-(U5-PA23-Pad32) -> /led4
Routing:
- net /led4: track 0.00 -> 88.2 mm, vias 0 -> 3
- net /led3: track 60.6 -> 110.1 mm
- net +5V: track 26.8 -> 54.9 mm, vias 19 -> 43
- net GND: track 110.6 -> 83.0 mm, vias 56 -> 45
- net /port2_isense2-: track 0.00 -> 27.2 mm, vias 0 -> 2
- net /port4_isense2-: track 0.00 -> 23.9 mm, vias 0 -> 2
- net /port3_isense1-: track 0.00 -> 23.7 mm, vias 0 -> 2
- net /port1_isense1-: track 0.00 -> 22.8 mm, vias 0 -> 2
- net /port3_isense2-: track 0.00 -> 20.9 mm
- net /port1_isense2-: track 0.00 -> 20.5 mm
- net /port1_isense1+: track 0.00 -> 19.0 mm, vias 0 -> 2
- net /port3_isense1+: track 0.00 -> 16.7 mm, vias 0 -> 2
- net /led1: track 43.6 -> 59.0 mm, vias 2 -> 3
- net /port1_isense2: track 14.8 -> 0.00 mm
- net +3V3: track 85.1 -> 71.0 mm, vias 17 -> 15
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Other:
- board size 100 x 50 mm -> 100 x 55 mm
