File: hardware/5v-power.kicad_sch (KiCad schematic)
At the start: 33 parts, among them J1 Conn_01x04, J2 Screw_Terminal_01x02, J8 Conn_01x03_Pin, J9 Conn_01x03_Pin, U2 INA4180, U3 INA4180, U4 AMS1117-3.3, U5 ATSAMD21G17A-M

Commit message: rev2
Parts:
- added D4: LED_Small, LED_SMD:LED_0603_1608Metric, symbol Device:LED_Small
- added R49: R_Small, Resistor_SMD:R_0603_1608Metric, symbol Device:R_Small
Connections:
- net port1_isense1 is gone; now on net port2_isense2+: U2.5 (IN+2)
- net port1_isense2 is gone; now on net port2_isense1+: U2.3 (IN+1)
- net port3_isense1 is gone; now on net port4_isense2+: U3.5 (IN+2)
- net port3_isense2 is gone; now on net port4_isense1+: U3.3 (IN+1)
- net GND: now also R49.2; no longer U2.13 (IN-4), U2.2 (IN-1), U2.6 (IN-2), U2.9 (IN-3), U3.13 (IN-4), U3.2 (IN-1), U3.6 (IN-2), U3.9 (IN-3)
- net port1_isense1_out: now also U2.14 (OUT4); no longer U2.7 (OUT2)
- net port1_isense2_out: now also U2.8 (OUT3); no longer U2.1 (OUT1)
- net port2_isense1+: no longer U2.12 (IN+4)
- net port2_isense1_out: now also U2.7 (OUT2); no longer U2.14 (OUT4)
- net port2_isense2+: no longer U2.10 (IN+3)
- net port2_isense2_out: now also U2.1 (OUT1); no longer U2.8 (OUT3)
- net port3_isense1_out: now also U3.14 (OUT4); no longer U3.7 (OUT2)
- net port3_isense2_out: now also U3.8 (OUT3); no longer U3.1 (OUT1)
- net port4_isense1+: no longer U3.12 (IN+4)
- net port4_isense1_out: now also U3.7 (OUT2); no longer U3.14 (OUT4)
- net port4_isense2+: no longer U3.10 (IN+3)
- net port4_isense2_out: now also U3.1 (OUT1); no longer U3.8 (OUT3)
- net led4: now reaches U5.32 (PA23)
- net led4: now also D4.2 (A)
- new net: D4.1 (K), R49.1
- new net port1_isense1+: U2.10 (IN+3)
- new net port1_isense1-: U2.9 (IN-3)
- new net port1_isense2+: U2.12 (IN+4)
- new net port1_isense2-: U2.13 (IN-4)
- new net port2_isense1-: U2.2 (IN-1)
- new net port2_isense2-: U2.6 (IN-2)
- new net port3_isense1+: U3.10 (IN+3)
- new net port3_isense1-: U3.9 (IN-3)
- new net port3_isense2+: U3.12 (IN+4)
- new net port3_isense2-: U3.13 (IN-4)
- new net port4_isense1-: U3.2 (IN-1)
- new net port4_isense2-: U3.6 (IN-2)
Other:
- sheet Port1 ports: added Isense_1-, Isense_2-; removed none
- sheet Port2 ports: added Isense_1-, Isense_2-; removed none
- sheet Port3 ports: added Isense_1-, Isense_2-; removed none
- sheet Port4 ports: added Isense_1-, Isense_2-; removed none
- note removed: "TODO * back usb port maybe idfk for samd flashing * samd swd * led placement - port leds? * make sure i have all the parts! even the weird ones!"
