File: hardware/ethernet.kicad_sch (KiCad schematic)
At the start: 25 parts, among them J7 RJ45_Abracon_ARJM11D7-009-AB-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, U1 W5500, Y1 RH100-25.000-18-F-1020-EXT-TR

Commit message: rev2
Parts:
- renumbered C12 to C11, C11 to C12
Changed lines of the file:
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@@
   (symbol (lib_id "power:GND") (at 102.87 128.905 0) (unit 1)
     (in_bom yes) (on_board yes) (dnp no) (fields_autoplaced)
-    (property "Reference" "#PWR010" (at 102.87 135.255 0)
+    (property "Reference" "#PWR066" (at 102.87 135.255 0)
       (effects (font (size 1.27 1.27)) hide)
     )
@@
     (instances
       (project "5v-power"
-        (path "/d0d0cd4d-faa1-43ba-b091-667ba93b62b4"
-          (reference "#PWR010") (unit 1)
-        )
         (path "/d0d0cd4d-faa1-43ba-b091-667ba93b62b4/7740e8c2-7d9b-470b-99d5-7c73dc6277d0"
           (reference "#PWR066") (unit 1)
@@
   (symbol (lib_id "power:+3V3") (at 97.79 67.945 0) (unit 1)
     (in_bom yes) (on_board yes) (dnp no) (fields_autoplaced)
-    (property "Reference" "#PWR060" (at 97.79 71.755 0)
+    (property "Reference" "#PWR064" (at 97.79 71.755 0)
       (effects (font (size 1.27 1.27)) hide)
     )
@@
     (instances
       (project "5v-power"
-        (path "/d0d0cd4d-faa1-43ba-b091-667ba93b62b4"
-          (reference "#PWR060") (unit 1)
-        )
         (path "/d0d0cd4d-faa1-43ba-b091-667ba93b62b4/7740e8c2-7d9b-470b-99d5-7c73dc6277d0"
           (reference "#PWR064") (unit 1)
@@
     (instances
       (project "5v-power"
-        (path "/d0d0cd4d-faa1-43ba-b091-667ba93b62b4"
-          (reference "C10") (unit 1)
-        )
         (path "/d0d0cd4d-faa1-43ba-b091-667ba93b62b4/7740e8c2-7d9b-470b-99d5-7c73dc6277d0"
           (reference "C10") (unit 1)
@@
   (symbol (lib_id "power:GND") (at 120.015 128.905 0) (unit 1)
     (in_bom yes) (on_board yes) (dnp no) (fields_autoplaced)
-    (property "Reference" "#PWR061" (at 120.015 135.255 0)
+    (property "Reference" "#PWR067" (at 120.015 135.255 0)
       (effects (font (size 1.27 1.27)) hide)
     )
@@
     (instances
       (project "5v-power"
-        (path "/d0d0cd4d-faa1-43ba-b091-667ba93b62b4"
-          (reference "#PWR061") (unit 1)
-        )
         (path "/d0d0cd4d-faa1-43ba-b091-667ba93b62b4/7740e8c2-7d9b-470b-99d5-7c73dc6277d0"
           (reference "#PWR067") (unit 1)
@@
     (instances
       (project "5v-power"
-        (path "/d0d0cd4d-faa1-43ba-b091-667ba93b62b4"
+        (path "/d0d0cd4d-faa1-43ba-b091-667ba93b62b4/7740e8c2-7d9b-470b-99d5-7c73dc6277d0"
           (reference "#PWR059") (unit 1)
         )
-        (path "/d0d0cd4d-faa1-43ba-b091-667ba93b62b4/7740e8c2-7d9b-470b-99d5-7c73dc6277d0"
-          (reference "#PWR059") (unit 1)
-        )
       )
     )
@@
     (instances
       (project "5v-power"
-        (path "/d0d0cd4d-faa1-43ba-b091-667ba93b62b4"
+        (path "/d0d0cd4d-faa1-43ba-b091-667ba93b62b4/7740e8c2-7d9b-470b-99d5-7c73dc6277d0"
           (reference "C4") (unit 1)
         )
-        (path "/d0d0cd4d-faa1-43ba-b091-667ba93b62b4/7740e8c2-7d9b-470b-99d5-7c73dc6277d0"
-          (reference "C4") (unit 1)
-        )
       )
     )
@@
   (symbol (lib_id "power:GND") (at 132.08 126.365 0) (unit 1)
     (in_bom yes) (on_board yes) (dnp no) (fields_autoplaced)
-    (property "Reference" "#PWR062" (at 132.08 132.715 0)
+    (property "Reference" "#PWR068" (at 132.08 132.715 0)
       (effects (font (size 1.27 1.27)) hide)
     )
@@
     (instances
       (project "5v-power"
-        (path "/d0d0cd4d-faa1-43ba-b091-667ba93b62b4"
-          (reference "#PWR062") (unit 1)
-        )
         (path "/d0d0cd4d-faa1-43ba-b091-667ba93b62b4/7740e8c2-7d9b-470b-99d5-7c73dc6277d0"
           (reference "#PWR068") (unit 1)
@@
     (instances
       (project "5v-power"
-        (path "/d0d0cd4d-faa1-43ba-b091-667ba93b62b4"
+        (path "/d0d0cd4d-faa1-43ba-b091-667ba93b62b4/7740e8c2-7d9b-470b-99d5-7c73dc6277d0"
           (reference "U1") (unit 1)
         )
-        (path "/d0d0cd4d-faa1-43ba-b091-667ba93b62b4/7740e8c2-7d9b-470b-99d5-7c73dc6277d0"
-          (reference "U1") (unit 1)
-        )
       )
     )
@@
     (instances
       (project "5v-power"
-        (path "/d0d0cd4d-faa1-43ba-b091-667ba93b62b4"
+        (path "/d0d0cd4d-faa1-43ba-b091-667ba93b62b4/7740e8c2-7d9b-470b-99d5-7c73dc6277d0"
           (reference "#PWR063") (unit 1)
         )
-        (path "/d0d0cd4d-faa1-43ba-b091-667ba93b62b4/7740e8c2-7d9b-470b-99d5-7c73dc6277d0"
-          (reference "#PWR063") (unit 1)
-        )
       )
     )
@@
     (instances
       (project "5v-power"
-        (path "/d0d0cd4d-faa1-43ba-b091-667ba93b62b4"
+        (path "/d0d0cd4d-faa1-43ba-b091-667ba93b62b4/7740e8c2-7d9b-470b-99d5-7c73dc6277d0"
           (reference "FB1") (unit 1)
         )
-        (path "/d0d0cd4d-faa1-43ba-b091-667ba93b62b4/7740e8c2-7d9b-470b-99d5-7c73dc6277d0"
-          (reference "FB1") (unit 1)
-        )
       )
     )
@@
     (instances
       (project "5v-power"
-        (path "/d0d0cd4d-faa1-43ba-b091-667ba93b62b4"
+        (path "/d0d0cd4d-faa1-43ba-b091-667ba93b62b4/7740e8c2-7d9b-470b-99d5-7c73dc6277d0"
           (reference "R33") (unit 1)
         )
-        (path "/d0d0cd4d-faa1-43ba-b091-667ba93b62b4/7740e8c2-7d9b-470b-99d5-7c73dc6277d0"
-          (reference "R33") (unit 1)
-        )
       )
     )
@@
     (instances
       (project "5v-power"
-        (path "/d0d0cd4d-faa1-43ba-b091-667ba93b62b4"
-          (reference "#PWR058") (unit 1)
-        )
         (path "/d0d0cd4d-faa1-43ba-b091-667ba93b62b4/7740e8c2-7d9b-470b-99d5-7c73dc6277d0"
           (reference "#PWR058") (unit 1)
@@
   (symbol (lib_id "Device:C_Small") (at 132.08 123.825 0) (unit 1)
     (in_bom yes) (on_board yes) (dnp no) (fields_autoplaced)
-    (property "Reference" "C11" (at 134.62 122.5613 0)
+    (property "Reference" "C12" (at 134.62 122.5613 0)
       (effects (font (size 1.27 1.27)) (justify left))
     )
@@
     (instances
       (project "5v-power"
-        (path "/d0d0cd4d-faa1-43ba-b091-667ba93b62b4"
-          (reference "C11") (unit 1)
-        )
         (path "/d0d0cd4d-faa1-43ba-b091-667ba93b62b4/7740e8c2-7d9b-470b-99d5-7c73dc6277d0"
           (reference "C12") (unit 1)
@@
   (symbol (lib_id "Device:C_Small") (at 120.015 126.365 0) (unit 1)
     (in_bom yes) (on_board yes) (dnp no) (fields_autoplaced)
-    (property "Reference" "C12" (at 123.19 125.1013 0)
+    (property "Reference" "C11" (at 123.19 125.1013 0)
       (effects (font (size 1.27 1.27)) (justify left))
     )
@@
     (instances
       (project "5v-power"
-        (path "/d0d0cd4d-faa1-43ba-b091-667ba93b62b4"
-          (reference "C12") (unit 1)
-        )
         (path "/d0d0cd4d-faa1-43ba-b091-667ba93b62b4/7740e8c2-7d9b-470b-99d5-7c73dc6277d0"
           (reference "C11") (unit 1)
@@
   (symbol (lib_id "power:GND") (at 140.97 121.285 0) (unit 1)
     (in_bom yes) (on_board yes) (dnp no) (fields_autoplaced)
-    (property "Reference" "#PWR011" (at 140.97 127.635 0)
+    (property "Reference" "#PWR069" (at 140.97 127.635 0)
       (effects (font (size 1.27 1.27)) hide)
     )
@@
     (instances
       (project "5v-power"
-        (path "/d0d0cd4d-faa1-43ba-b091-667ba93b62b4"
-          (reference "#PWR011") (unit 1)
-        )
         (path "/d0d0cd4d-faa1-43ba-b091-667ba93b62b4/7740e8c2-7d9b-470b-99d5-7c73dc6277d0"
           (reference "#PWR069") (unit 1)
@@
   (symbol (lib_id "power:GND") (at 97.79 128.905 0) (unit 1)
     (in_bom yes) (on_board yes) (dnp no) (fields_autoplaced)
-    (property "Reference" "#PWR07" (at 97.79 135.255 0)
+    (property "Reference" "#PWR065" (at 97.79 135.255 0)
       (effects (font (size 1.27 1.27)) hide)
     )
@@
     (instances
       (project "5v-power"
-        (path "/d0d0cd4d-faa1-43ba-b091-667ba93b62b4"
-          (reference "#PWR07") (unit 1)
-        )
         (path "/d0d0cd4d-faa1-43ba-b091-667ba93b62b4/7740e8c2-7d9b-470b-99d5-7c73dc6277d0"
           (reference "#PWR065") (unit 1)
